Commit message: Show the D435i and mount bracket in the web robot viewer
- gen_robot_model_assets.py emits camera + bracket links/joints, reading
  camera.yaml and go2_sim.camera_geometry from the outer repo
- The viewer has no TF, so the camera is joined into the URDF directly
- Primitives not a mesh (Intel's d435.dae is 231k triangles); urdf-loader
  draws box/cylinder natively, so robot_viewer.js is unchanged
- Same block applied to the vendored go2.urdf, since regenerating needs
  pycollada; --no-camera omits it

File: src/go2_remote_controller/app/static/robot_model/go2.urdf (robot description, URDF)
Before this commit: robot go2, 31 links, 30 joints
Links:
- added link camera_link; visual box size=0.002000 0.086000 0.021000; visual box size=0.012000 0.020000 0.004000
- added link camera_mount; visual box size=0.014000 0.030000 0.100000; visual box size=0.120000 0.030000 0.010000
Joints:
- added joint camera_link_joint: type fixed, parent base_link, child camera_link, origin xyz=0.280000 0.000000 0.100000 rpy=0.000000 0.523599 0.000000
- added joint camera_mount_joint: type fixed, parent base_link, child camera_mount, origin xyz=0 0 0 rpy=0 0 0
